Commit message: Fix MISUMI catalog mismatches found by cross-checking misumi-ec.com
Cross-checked every catalogue part against kr.misumi-ec.com:
- SHF20: catalogue T=20 is the overall axial length including the
  8 mm flange; the model used 8 + 20 = 28. Boss is now 12, flange height
  A34. Stack-up shrinks by 8, rocker shaft SF 4.15 -> 4.86.
- Set collar: "SCS20" on MISUMI is a third-party shackle. The collar is
  PSCS20-12 (ID 20 / OD 40 / W 12); model OD 32 -> 40.
- Upper arm rails: HFS5-3030 does not exist; 30x30 is HFS6-3030
  (A 333 mm2, I 2.83e4, 0.9 kg/m). Renamed; section values updated.
- Series-5 slot T-nuts (HNTT5/HNTP5) are M3-M5 only, and HFS5-4040 has
  two slots per face at +-10. Bolt holes were on face centres or off
  the profile:
  * SHF20 bolts sat between the side rail's slots -> lower rail centre
    300 -> 310 so its lower slot is at the pivot height (Z 300);
    ground clearance 280 -> 290. SHF20 dia 7 holes take M5.
  * J1 base plate M8 at rail/crossmember centres -> M5 on the slot lines.
  * Differential post M8 at X +-30 (outside the 40 mm crossmember) ->
    4x M5 on the crossmember slots.
- arm_check: forearm deflection used an extrusion section, the forearm
  is an Al tube 50x2 -> tip deflection 1.14 -> 0.62 mm (bracket share 9%).
- Verified as listed: SFJ12/16/20 (SUJ2), B6001/6002/6004/6810/6811/6813
  ZZ, PHS8 (Ozak/TRUSCO), IKO CRBH8016A cross roller, HFS5-4040.
- Gas spring: no MISUMI FGSS size fits the 174-279 mm (ratio 1.6) range
  of the current r100/h180 geometry; recorded as an open item.
- tests: SHF20 length, holder bolts on rail slot, base plate and post
  bolts on slot lines (66 pass). Regenerated suspension/robot/URDF/DXF
  outputs and .f3d; track 1032 -> 1016.

Co-Authored-By: Claude Opus 5.5 <noreply@anthropic.com>

File: output/urdf/orchard_rover_description/urdf/orchard_rover.urdf (robot description, URDF)
Before this commit: robot orchard_rover, 8 links, 7 joints
Links:
- link base_link: mass 124.730443 -> 124.523125

Commit message: J2 gas spring: MISUMI FGSS22120C with re-placed anchors
The previous balancer (r100 / h180, 350 N) needed a 174-279 mm spring
(length ratio 1.6); no MISUMI gas spring fits (FGSS forces are 49-490 N
in steps, stroke 100 already starts at 286 mm). Searched all 17 FGSS
sizes against every mountable anchor position and picked FGSS22120C
(stroke 120, 320-440 mm, 392 N @ Lmax-10, dia 22):

- Base anchor at arm-frame (-35, -150): clevis 50 above the J1 turret.
- Arm anchor r280 / +10 deg on the J2 side plate (X 276, Z 49); the J2
  side plate is extended from X 210 to 285 (5 mm short of the J3 plate),
  with an extra rail bolt pair at X 240.
- Over the full J2 range (-20..90 deg) the spring stays at 327-434 mm
  (7 / 6 mm from the ends) and the J2 actuator demand, worst of arm
  extended+tool and folded without tool, x1.5, peaks at 65.3 N.m @ 31 deg
  (80 available; 120 without a spring).
- shoulder_joint: GasSpringSpec (catalogue data, assumed +30 % force
  progression), gas_spring_state / gas_spring_balance evaluate the whole
  angle range; torque_static 72.8 -> 79.7 to match arm_check.
- base_joint, transport_check, arm_check use the new anchors (J1 bracket
  SF 70 with the spring reaction).
- tests: catalogue length margins, actuator demand over the full range,
  gravity torque consistent with arm_check (67 pass). Motion and
  interference results unchanged; transport min clearance 72.1 mm.
- Regenerated arm/robot/shoulder/URDF/DXF outputs, PNGs, .f3d; docs.

Co-Authored-By: Claude Opus 5.5 <noreply@anthropic.com>

File: output/urdf/orchard_rover_description/urdf/orchard_rover.urdf (robot description, URDF)
Before this commit: robot orchard_rover, 8 links, 7 joints
Links:
- link j1_link: mass 5.89811828 -> 5.92144628
- link upper_arm: mass 4.57786638 -> 4.91584945

Commit message: Frame: separate MISUMI HFS5-4040 profile members with butt joints
The frame was a single fused block of 40x40 solid bars (a reference for
the suspension mounting points). It is now built from catalogue profile
members:

- hfs5_4040_section(): 40x40 with two slots per face at +-10 (opening 6)
  and the four dia 4.2 corner holes from the MISUMI drawing; T-slot
  interior and centre cavity approximated. Catalogue data (1.28 kg/m,
  A 472 mm2, I 8.89e4) is used for mass.
- frame_members(): side rails 1000 x4 run through; end cross members,
  differential cross member and J1 cross members (720 x7) butt against
  the rail inner faces; posts 350 x4 butt onto/under the rails. 15
  members, 10.44 m, 13.4 kg. Each member is its own body in the STEP.
- Joining: end tapping M5 in the corner holes + wrench holes in the
  through member (22 joints); no external brackets because the rail top
  and side faces carry the base plate, pivot holders and diff post.
- frame_cut_list.txt (output/robot) with lengths, quantities, joints.
- transport_check / test_motion use the per-member frame names.
- tests: members are single valid solids within catalogue length, no
  overlap, every butted member touches two others; the SHF20 bolt
  positions fall inside the rail slot openings (69 pass).
- Interference unchanged; combined arm-vehicle poses 30 -> 28 (slots
  remove 1 mm3 edge contacts). Regenerated outputs, URDF, .f3d.

Co-Authored-By: Claude Opus 5.5 <noreply@anthropic.com>

File: output/urdf/orchard_rover_description/urdf/orchard_rover.urdf (robot description, URDF)
Before this commit: robot orchard_rover, 8 links, 7 joints
Links:
- link base_link: mass 124.523125 -> 95.6607583

Commit message: Idler wheels: SFJ20 axle clamped by SHF20 holder, retained by PSCS20-12
The idler spec said 6003ZZ (bore 17) while the axle was Ø16, and the stub
axle only sat in a clearance hole in the bogie plate with nothing clamping
it or keeping the wheel on.

- Axle Ø16 -> SFJ20, hub bearing bore 20 (modelled 6004ZZ x2 in pockets)
- SHF20 holder on the bogie plate outer face, rotated 90° so the bolt row is
  vertical and the wheel-load moment goes into M6 bolt tension (plate tapped)
- Stack: plate | holder T20 | spacer 4 | wheel 80 | washer 2 | PSCS20-12
- wheel_gap 16 -> 24 for the holder; track 1016 -> 1032
- New SF: idler_axle 8.7, idler_holder_bolt 22.9; front axle 2.72 -> 2.62
- Tests for the retention stack; 71 pass. Fusion interference unchanged.

Co-Authored-By: Claude Opus 5.5 <noreply@anthropic.com>

File: output/urdf/orchard_rover_description/urdf/orchard_rover.urdf (robot description, URDF)
Before this commit: robot orchard_rover, 8 links, 7 joints
Links:
- link base_link: mass 95.6607583 -> 96.0805113

Commit message: Rocker/bogie/diff pivots: bolted MISUMI BGRBB holders replace integral bosses
The rocker plate, bogie plate and diff bar carried integral bearing bosses
that could not be cut from 12t plate. They are now single-thickness plates
(waterjet + taps) with commercial flanged holder sets bolted on:

- Rocker pivot: BGRBB6004DD-40 (M6 x4), flange on plate inner face
- Bogie pivot: BGRBB6001DD-25 (M4 x4), flange on plate outer face
- Diff bar: BGRBB6001DD-25 (M4 x4) on a center pad, new diff_bar.dxf

Inner-ring spacers locate each bearing axially and keep the rotating holders
clear of SHF20, the shaft collar, the rocker plate and the diff post.
plate_gap 6 -> 8; track 1032 -> 1058, overall width 1182. Rocker shaft SF
4.0, tip-over margins 4.48 / 1.99, combined arm collisions 27. BOM
~1,102,000 KRW. New tests check plates have no bosses and that holders,
bearings and spacers seat without overlap.

Co-Authored-By: Claude Opus 5.5 <noreply@anthropic.com>

File: output/urdf/orchard_rover_description/urdf/orchard_rover.urdf (robot description, URDF)
Before this commit: robot orchard_rover, 8 links, 7 joints
Links:
- link base_link: mass 96.0805113 -> 96.3148933

Commit message: Bogie shaft: PSCS12-10 collar retains the bogie group outboard
The SFJ12 bogie shaft is pressed into the rocker plate, but nothing held the
bogie holder/bearings on its outer end (only a 10 mm "retaining ring"
allowance). Add an inner-ring spacer (Ø16, l + 1) from the outer 6001 to
1 mm past the holder flange and a MISUMI PSCS12-10 slit collar (OD 30,
width 10, checked on misumi-ec.com). Shaft 50 -> 53; its end stays 3 mm
inside the middle wheel. make_shaft_collar takes bore/od/width.

Test chain extended to rocker_plate | spacer | 6001 x2 | spacer | collar,
with holder-collar clearance and wheel clearance. Interference unchanged
(Fusion 10 pairs, 10518.3 mm3). BOM ~1,116,000 KRW.

Co-Authored-By: Claude Opus 5.5 <noreply@anthropic.com>

File: output/urdf/orchard_rover_description/urdf/orchard_rover.urdf (robot description, URDF)
Before this commit: robot orchard_rover, 8 links, 7 joints
Links:
- link base_link: mass 96.3148933 -> 96.3505892

Commit message: Diff pin: STWN12 snap ring retains the diff bar on its pivot pin
The diff bar holder sat on the post pin with only a 4 mm "retaining ring
allowance" above it, so nothing kept the bar from lifting off. Add an
inner-ring spacer (Ø16, l + 1) from the upper 6001 to 1 mm above the holder
and a MISUMI STWN12 shaft C-ring (t 1) in a Ø11.5 x 1.15 groove cut in the
pin. The pin top stays 4 mm above the holder.

A PSCS12-10 collar was tried first, but the 9 mm longer pin hit the J4
housing with the arm folded rearward (J1 ±180, J2 0, J3 -120), raising
combined collisions 27 -> 29. With the snap ring they stay at 27.

Test chain extended to post | spacer | 6001 x2 | spacer | ring | post, plus
ring-holder clearance and pin height. Interference unchanged (Fusion 10
pairs, 10518.3 mm3). BOM ~1,117,000 KRW.

Co-Authored-By: Claude Opus 5.5 <noreply@anthropic.com>

File: output/urdf/orchard_rover_description/urdf/orchard_rover.urdf (robot description, URDF)
Before this commit: robot orchard_rover, 8 links, 7 joints
Links:
- link base_link: mass 96.3505892 -> 96.3517132
